Commit message: flip Franka direction on summit

File: robot_description/mobile_franka.urdf (robot description, URDF)
Before this commit: robot summit_panda, 21 links, 20 joints
Joints:
- joint franka_fixed: origin xyz=0.0325484 0.0121688 0.0266862 rpy=0. 0. 0. -> xyz=-0.0325484 0 0.0266862 rpy=0. 0. 3.141592653589793
